File: pcb-lab-1.kicad_pcb (KiCad board)
At the start: 2 copper layers, 91.4 x 33 mm, 66 parts, among them J1 BAT, J10 JP_RX, J11 JP_TX, J14 JP_RX, J15 JP_TX, J18 UART, J2 UPDI_PIN_SMD, J20 UPDI, Q30 NMOS_GSD, Q31 NMOS_GSD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

Commit message: Silkscreen
Other:
- board text added: "(C) Vlad Belous CC BY-SA 4.0"
- board text added: "2V5"
- board text added: "5V"
- board text added: "74LVC"
- board text added: "G"
- board text added: "GND"
- board text added: "GRN"
- board text added: "I2C VBAT"
- board text added: "MOSFET"
- board text added: "NLSX"
- board text added: "Open-drain: NLSX4373 Push-pull auto: TXB0104, PI4ULS Push-pull dir: 74LVC1T45"
- board text added: "PCB Lab #1 Level Translation"
- board text added: "PI4ULS"
- board text added: "RED"
- board text added: "RX"
- board text added: "SCL"
- board text added: "SDA"
- board text added: "TX"
- board text added: "TXB"
- board text added: "UPDI"
- board text added: "UPDI 2V5"
- board text added: "UPDI 5V"
- board text added: "VBAT"
- board text added: "VBAT an.sw"
- board text added: "VBAT ap2280"
- board text added: "YEL"
- board text added: "analog"
Changed lines of the file:
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@@
   (general
     (thickness 1.6)
-    (drawings 17)
+    (drawings 77)
     (tracks 695)
     (zones 0)
@@
     (descr "Linx BAT-HLD-001-THM")
     (tags "Battery Holder CR2032 Linx BAT-HLD-001-THM")
-    (fp_text reference BT1 (at -5.842 -8.636 90) (layer F.SilkS)
+    (fp_text reference BT1 (at 5.686 -8.7 90) (layer F.SilkS)
       (effects (font (size 1 1) (thickness 0.15)))
     )
@@
     (tags resistor)
     (attr smd)
-    (fp_text reference R5 (at -2.3 0) (layer F.SilkS)
+    (fp_text reference R5 (at -1.9 -0.6) (layer F.SilkS)
       (effects (font (size 0.635 0.635) (thickness 0.127)))
     )
@@
     (tags SOT-23-6)
     (attr smd)
-    (fp_text reference U1 (at 0.1 2.4) (layer F.SilkS)
+    (fp_text reference U1 (at -1 -2.1) (layer F.SilkS)
       (effects (font (size 0.635 0.635) (thickness 0.127)))
     )
@@
     (tags "SOIC 1.27")
     (attr smd)
-    (fp_text reference U2 (at 0 -2.9 180) (layer F.SilkS)
+    (fp_text reference U2 (at -0.8 -3.1 180) (layer F.SilkS)
       (effects (font (size 0.762 0.762) (thickness 0.127)))
     )
@@
     (tags SOT-23-6)
     (attr smd)
-    (fp_text reference U5 (at 2.9 -0.2) (layer F.SilkS)
+    (fp_text reference U5 (at -1.8 -2.1) (layer F.SilkS)
       (effects (font (size 0.635 0.635) (thickness 0.127)))
     )
@@
     )
   )
+  (gr_text "Open-drain:\nNLSX4373\n\nPush-pull auto:\nTXB0104, PI4ULS\n\nPush-pull dir:\n74LVC1T45" (at 159.9 98.1) (layer B.SilkS)
+    (effects (font (size 1.016 1.016) (thickness 0.1524)) (justify left mirror))
+  )
+  (gr_text GND (at 122.1 81.3) (layer F.SilkS)
+    (effects (font (size 0.762 0.762) (thickness 0.1524)))
+  )
+  (gr_text "(C) Vlad Belous\nCC BY-SA 4.0" (at 143.6 80.1) (layer B.SilkS)
+    (effects (font (size 1.016 1.016) (thickness 0.1524)) (justify left mirror))
+  )
+  (gr_text "PCB Lab #1\nLevel Translation" (at 143.7 75.4) (layer B.SilkS)
+    (effects (font (size 1.016 1.016) (thickness 0.1524)) (justify left mirror))
+  )
+  (gr_text GRN (at 152.9 92.3) (layer F.SilkS)
+    (effects (font (size 0.762 0.762) (thickness 0.1524)))
+  )
+  (gr_text YEL (at 155.5 92.3) (layer F.SilkS)
+    (effects (font (size 0.762 0.762) (thickness 0.1524)))
+  )
+  (gr_text RED (at 158.1 92.3) (layer F.SilkS)
+    (effects (font (size 0.762 0.762) (thickness 0.1524)))
+  )
+  (gr_text UPDI (at 192.9 96.6) (layer B.SilkS)
+    (effects (font (size 0.762 0.762) (thickness 0.1524)) (justify mirror))
+  )
+  (gr_text GND (at 127 81.3) (layer B.SilkS)
+    (effects (font (size 0.762 0.762) (thickness 0.1524)) (justify mirror))
+  )
+  (gr_text VBAT (at 127.1 78.7) (layer B.SilkS)
+    (effects (font (size 0.762 0.762) (thickness 0.1524)) (justify mirror))
+  )
+  (gr_text SCL (at 127 76.2) (layer B.SilkS)
+    (effects (font (size 0.762 0.762) (thickness 0.1524)) (justify mirror))
+  )
+  (gr_text SDA (at 127 73.7) (layer B.SilkS)
+    (effects (font (size 0.762 0.762) (thickness 0.1524)) (justify mirror))
+  )
+  (gr_text TX (at 193.6 83.8) (layer B.SilkS)
+    (effects (font (size 0.762 0.762) (thickness 0.1524)) (justify mirror))
+  )
+  (gr_text RX (at 193.6 81.3) (layer B.SilkS)
+    (effects (font (size 0.762 0.762) (thickness 0.1524)) (justify mirror))
+  )
+  (gr_text G (at 193.7 78.7) (layer B.SilkS)
+    (effects (font (size 0.762 0.762) (thickness 0.1524)) (justify mirror))
+  )
+  (gr_text 5V (at 193.5 76.2) (layer B.SilkS)
+    (effects (font (size 0.762 0.762) (thickness 0.1524)) (justify mirror))
+  )
+  (gr_text G (at 193.5 94) (layer B.SilkS)
+    (effects (font (size 0.762 0.762) (thickness 0.1524)) (justify mirror))
+  )
+  (gr_text 5V (at 193.3 91.5) (layer B.SilkS)
+    (effects (font (size 0.762 0.762) (thickness 0.1524)) (justify mirror))
+  )
+  (gr_text GND (at 116.9 101.7) (layer B.SilkS)
+    (effects (font (size 0.762 0.762) (thickness 0.1524)) (justify mirror))
+  )
+  (gr_text VBAT (at 116.9 99.1) (layer B.SilkS)
+    (effects (font (size 0.762 0.762) (thickness 0.1524)) (justify mirror))
+  )
+  (gr_text "UPDI\n5V" (at 187.9 99.2) (layer F.SilkS)
+    (effects (font (size 0.762 0.762) (thickness 0.1524)))
+  )
+  (gr_text PI4ULS (at 184.7 96.6) (layer F.SilkS)
+    (effects (font (size 0.762 0.762) (thickness 0.1524)))
+  )
+  (gr_text TXB (at 185.7 91.5) (layer F.SilkS)
+    (effects (font (size 0.762 0.762) (thickness 0.1524)))
+  )
+  (gr_text UPDI (at 195 98.5) (layer F.SilkS)
+    (effects (font (size 0.762 0.762) (thickness 0.1524)))
+  )
+  (gr_text G (at 193.6 94) (layer F.SilkS)
+    (effects (font (size 0.762 0.762) (thickness 0.1524)))
+  )
+  (gr_text 5V (at 193.5 91.4) (layer F.SilkS)
+    (effects (font (size 0.762 0.762) (thickness 0.1524)))
+  )
+  (gr_text 5V (at 193.6 76.3) (layer F.SilkS)
+    (effects (font (size 0.762 0.762) (thickness 0.1524)))
+  )
+  (gr_text G (at 193.6 78.8) (layer F.SilkS)
+    (effects (font (size 0.762 0.762) (thickness 0.1524)))
+  )
+  (gr_text TX (at 193.7 84) (layer F.SilkS)
+    (effects (font (size 0.762 0.762) (thickness 0.1524)))
+  )
+  (gr_text RX (at 193.7 81.4) (layer F.SilkS)
+    (effects (font (size 0.762 0.762) (thickness 0.1524)))
+  )
+  (gr_text 74LVC (at 170.3 81.3) (layer F.SilkS)
+    (effects (font (size 0.635 0.635) (thickness 0.127)))
+  )
+  (gr_text 74LVC (at 182.7 81.3) (layer F.SilkS)
+    (effects (font (size 0.635 0.635) (thickness 0.127)))
+  )
+  (gr_text TXB (at 183.1 76.2) (layer F.SilkS)
+    (effects (font (size 0.762 0.762) (thickness 0.1524)))
+  )
+  (gr_text TXB (at 170 76.2) (layer F.SilkS)
+    (effects (font (size 0.762 0.762) (thickness 0.1524)))
+  )
+  (gr_text 5V (at 186.6 74.4) (layer F.SilkS)
+    (effects (font (size 0.762 0.762) (thickness 0.1524)))
+  )
+  (gr_text 2V5 (at 166.3 74.4) (layer F.SilkS)
+    (effects (font (size 0.762 0.762) (thickness 0.1524)))
+  )
+  (gr_text RX (at 167.7 83.1) (layer F.SilkS)
+    (effects (font (size 0.762 0.762) (thickness 0.1524)))
+  )
+  (gr_text RX (at 188 83.1) (layer F.SilkS)
+    (effects (font (size 0.762 0.762) (thickness 0.1524)))
+  )
+  (gr_text TX (at 185.5 83.1) (layer F.SilkS)
+    (effects (font (size 0.762 0.762) (thickness 0.1524)))
+  )
+  (gr_text TX (at 165.1 83.1) (layer F.SilkS)
+    (effects (font (size 0.762 0.762) (thickness 0.1524)))
+  )
+  (gr_text "UPDI\n2V5" (at 165.2 99.2) (layer F.SilkS)
+    (effects (font (size 0.762 0.762) (thickness 0.1524)))
+  )
+  (gr_text PI4ULS (at 168.3 96.8) (layer F.SilkS)
+    (effects (font (size 0.762 0.762) (thickness 0.1524)))
+  )
+  (gr_text TXB (at 167.4 91.3) (layer F.SilkS)
+    (effects (font (size 0.762 0.762) (thickness 0.1524)))
+  )
+  (gr_text "VBAT\nap2280" (at 155.1 90.2) (layer F.SilkS)
+    (effects (font (size 0.762 0.762) (thickness 0.1524)))
+  )
+  (gr_text "VBAT\nan.sw" (at 150 90.2) (layer F.SilkS)
+    (effects (font (size 0.762 0.762) (thickness 0.1524)))
+  )
+  (gr_text analog (at 141.9 84.7) (layer F.SilkS)
+    (effects (font (size 0.762 0.762) (thickness 0.1524)))
+  )
+  (gr_text VBAT (at 121.9 78.7) (layer F.SilkS)
+    (effects (font (size 0.762 0.762) (thickness 0.1524)))
+  )
+  (gr_text SCL (at 122 76.1) (layer F.SilkS)
+    (effects (font (size 0.762 0.762) (thickness 0.1524)))
+  )
+  (gr_text SDA (at 122 73.6) (layer F.SilkS)
+    (effects (font (size 0.762 0.762) (thickness 0.1524)))
+  )
+  (gr_text GND (at 116.8 101.7) (layer F.SilkS)
+    (effects (font (size 0.762 0.762) (thickness 0.1524)))
+  )
+  (gr_text VBAT (at 116.9 99.1) (layer F.SilkS)
+    (effects (font (size 0.762 0.762) (thickness 0.1524)))
+  )
+  (gr_text MOSFET (at 148.5 100.3) (layer F.SilkS)
+    (effects (font (size 0.889 0.889) (thickness 0.1524)))
+  )
+  (gr_text "NLSX\n" (at 147.8 97.7) (layer F.SilkS)
+    (effects (font (size 0.889 0.889) (thickness 0.1524)))
+  )
+  (gr_text SDA (at 145 103.7) (layer F.SilkS)
+    (effects (font (size 0.889 0.889) (thickness 0.1524)))
+  )
+  (gr_text SCL (at 142.2 103.7) (layer F.SilkS)
+    (effects (font (size 0.889 0.889) (thickness 0.1524)))
+  )
+  (gr_text SCL (at 127.1 103.7) (layer F.SilkS)
+    (effects (font (size 0.889 0.889) (thickness 0.1524)))
+  )
+  (gr_text SDA (at 124.3 103.7) (layer F.SilkS)
+    (effects (font (size 0.889 0.889) (thickness 0.1524)))
+  )
+  (gr_text MOSFET (at 120.7 100.3) (layer F.SilkS)
+    (effects (font (size 0.889 0.889) (thickness 0.1524)))
+  )
+  (gr_text "NLSX\n" (at 121.3 97.7) (layer F.SilkS)
+    (effects (font (size 0.889 0.889) (thickness 0.1524)))
+  )
+  (gr_text "I2C\nVBAT" (at 125.9 93.8) (layer F.SilkS)
+    (effects (font (size 1 1) (thickness 0.15)))
+  )
   (gr_line (start 106.68 66.04) (end 106.68 71.12) (layer Cmts.User) (width 0.15))
